File: light sensitive demo.sch (KiCad schematic (older format))
At the start: 8 parts, among them U1 LM321

Commit message: Changed adjustment potentiometer to push-button
Parts:
- removed RV1: R_POT, symbol Device:R_POT
- added Q?: IRF3205, Package_TO_SOT_THT:TO-220-3_Vertical, symbol Transistor_FET:IRF3205
- added SW?: SW_Push_Dual, symbol Switch:SW_Push_Dual
- R2: value R -> 5k1
- R3: value R -> 330
Other:
- moved on the sheet: D1
Changed lines of the file:
@@
 EESchema Schematic File Version 4
+LIBS:light sensitive demo-cache
 EELAYER 26 0
 EELAYER END
@@
 L Diode:1N4006 D1
 U 1 1 5B7F9684
-P 4250 3500
-F 0 "D1" H 4250 3716 50  0000 C CNN
-F 1 "1N4006" H 4250 3625 50  0000 C CNN
-F 2 "Diode_THT:D_DO-41_SOD81_P10.16mm_Horizontal" H 4250 3325 50  0001 C CNN
-F 3 "http://www.vishay.com/docs/88503/1n4001.pdf" H 4250 3500 50  0001 C CNN
-	1    4250 3500
+P 3800 3500
+F 0 "D1" H 3800 3716 50  0000 C CNN
+F 1 "1N4006" H 3800 3625 50  0000 C CNN
+F 2 "Diode_THT:D_DO-41_SOD81_P10.16mm_Horizontal" H 3800 3325 50  0001 C CNN
+F 3 "http://www.vishay.com/docs/88503/1n4001.pdf" H 3800 3500 50  0001 C CNN
+	1    3800 3500
 	1    0    0    -1
 $EndComp
@@
 L power:GND #PWR0101
 U 1 1 5B7FA197
-P 4500 3900
-F 0 "#PWR0101" H 4500 3650 50  0001 C CNN
-F 1 "GND" H 4505 3727 50  0000 C CNN
-F 2 "" H 4500 3900 50  0001 C CNN
-F 3 "" H 4500 3900 50  0001 C CNN
-	1    4500 3900
+P 4050 3900
+F 0 "#PWR0101" H 4050 3650 50  0001 C CNN
+F 1 "GND" H 4055 3727 50  0000 C CNN
+F 2 "" H 4050 3900 50  0001 C CNN
+F 3 "" H 4050 3900 50  0001 C CNN
+	1    4050 3900
 	1    0    0    -1
 $EndComp
@@
 L Device:R_PHOTO R1
 U 1 1 5B7FA4F4
-P 3550 3350
-F 0 "R1" H 3620 3396 50  0000 L CNN
-F 1 "R_PHOTO" H 3620 3305 50  0000 L CNN
-F 2 "" V 3600 3100 50  0001 L CNN
-F 3 "~" H 3550 3300 50  0001 C CNN
-	1    3550 3350
+P 3100 3350
+F 0 "R1" H 3170 3396 50  0000 L CNN
+F 1 "R_PHOTO" H 3170 3305 50  0000 L CNN
+F 2 "" V 3150 3100 50  0001 L CNN
+F 3 "~" H 3100 3300 50  0001 C CNN
+	1    3100 3350
 	1    0    0    -1
 $EndComp
@@
 L Device:CP C1
 U 1 1 5B7FA748
-P 4500 3750
-F 0 "C1" H 4618 3796 50  0000 L CNN
-F 1 "CP" H 4618 3705 50  0000 L CNN
-F 2 "" H 4538 3600 50  0001 C CNN
-F 3 "~" H 4500 3750 50  0001 C CNN
-	1    4500 3750
-	1    0    0    -1
-$EndComp
-$Comp
-L Device:R_POT RV1
-U 1 1 5B7FA853
-P 3900 4550
-F 0 "RV1" H 3830 4596 50  0000 R CNN
-F 1 "R_POT" H 3830 4505 50  0000 R CNN
-F 2 "" H 3900 4550 50  0001 C CNN
-F 3 "~" H 3900 4550 50  0001 C CNN
-	1    3900 4550
-	1    0    0    -1
-$EndComp
-$Comp
-L power:GND #PWR0102
-U 1 1 5B7FAA51
-P 3900 4700
-F 0 "#PWR0102" H 3900 4450 50  0001 C CNN
-F 1 "GND" H 3905 4527 50  0000 C CNN
-F 2 "" H 3900 4700 50  0001 C CNN
-F 3 "" H 3900 4700 50  0001 C CNN
-	1    3900 4700
+P 4050 3750
+F 0 "C1" H 4168 3796 50  0000 L CNN
+F 1 "CP" H 4168 3705 50  0000 L CNN
+F 2 "" H 4088 3600 50  0001 C CNN
+F 3 "~" H 4050 3750 50  0001 C CNN
+	1    4050 3750
 	1    0    0    -1
 $EndComp
@@
 L Device:R R2
 U 1 1 5B7FABD0
-P 3550 3650
-F 0 "R2" H 3620 3696 50  0000 L CNN
-F 1 "R" H 3620 3605 50  0000 L CNN
-F 2 "" V 3480 3650 50  0001 C CNN
-F 3 "~" H 3550 3650 50  0001 C CNN
-	1    3550 3650
+P 3100 3650
+F 0 "R2" H 3170 3696 50  0000 L CNN
+F 1 "5k1" H 3170 3605 50  0000 L CNN
+F 2 "" V 3030 3650 50  0001 C CNN
+F 3 "~" H 3100 3650 50  0001 C CNN
+	1    3100 3650
 	1    0    0    -1
 $EndComp
@@
 L power:GND #PWR0103
 U 1 1 5B7FAC69
-P 3550 3800
-F 0 "#PWR0103" H 3550 3550 50  0001 C CNN
-F 1 "GND" H 3555 3627 50  0000 C CNN
-F 2 "" H 3550 3800 50  0001 C CNN
-F 3 "" H 3550 3800 50  0001 C CNN
-	1    3550 3800
-	1    0    0    -1
-$EndComp
-Wire Wire Line
-	4400 3500 4500 3500
-Wire Wire Line
-	4500 3500 4500 3600
-Wire Wire Line
-	4500 3500 5050 3500
-Connection ~ 4500 3500
-Wire Wire Line
-	5050 3700 4900 3700
-Wire Wire Line
-	4900 3700 4900 4550
-Wire Wire Line
-	4100 3500 3550 3500
-Connection ~ 3550 3500
-Wire Wire Line
-	4050 4550 4900 4550
+P 3100 3800
+F 0 "#PWR0103" H 3100 3550 50  0001 C CNN
+F 1 "GND" H 3105 3627 50  0000 C CNN
+F 2 "" H 3100 3800 50  0001 C CNN
+F 3 "" H 3100 3800 50  0001 C CNN
+	1    3100 3800
+	1    0    0    -1
+$EndComp
+Wire Wire Line
+	3950 3500 4050 3500
+Wire Wire Line
+	4050 3500 4050 3600
+Connection ~ 4050 3500
+Connection ~ 3100 3500
 $Comp
 L Device:LED D2
@@
 P 5950 3750
 F 0 "R3" H 6020 3796 50  0000 L CNN
-F 1 "R" H 6020 3705 50  0000 L CNN
+F 1 "330" H 6020 3705 50  0000 L CNN
 F 2 "" V 5880 3750 50  0001 C CNN
 F 3 "~" H 5950 3750 50  0001 C CNN
@@
 L power:VCC #PWR0105
 U 1 1 5B7FB948
-P 3550 3200
-F 0 "#PWR0105" H 3550 3050 50  0001 C CNN
-F 1 "VCC" H 3567 3373 50  0000 C CNN
-F 2 "" H 3550 3200 50  0001 C CNN
-F 3 "" H 3550 3200 50  0001 C CNN
-	1    3550 3200
-	1    0    0    -1
-$EndComp
-$Comp
-L power:VCC #PWR0106
-U 1 1 5B7FB981
-P 3900 4400
-F 0 "#PWR0106" H 3900 4250 50  0001 C CNN
-F 1 "VCC" H 3917 4573 50  0000 C CNN
-F 2 "" H 3900 4400 50  0001 C CNN
-F 3 "" H 3900 4400 50  0001 C CNN
-	1    3900 4400
+P 3100 3200
+F 0 "#PWR0105" H 3100 3050 50  0001 C CNN
+F 1 "VCC" H 3117 3373 50  0000 C CNN
+F 2 "" H 3100 3200 50  0001 C CNN
+F 3 "" H 3100 3200 50  0001 C CNN
+	1    3100 3200
 	1    0    0    -1
 $EndComp
@@
 L power:PWR_FLAG #FLG0101
 U 1 1 5B7FBBDE
-P 5450 4700
-F 0 "#FLG0101" H 5450 4775 50  0001 C CNN
-F 1 "PWR_FLAG" H 5450 4874 50  0000 C CNN
-F 2 "" H 5450 4700 50  0001 C CNN
-F 3 "~" H 5450 4700 50  0001 C CNN
-	1    5450 4700
+P 6600 5000
+F 0 "#FLG0101" H 6600 5075 50  0001 C CNN
+F 1 "PWR_FLAG" H 6600 5174 50  0000 C CNN
+F 2 "" H 6600 5000 50  0001 C CNN
+F 3 "~" H 6600 5000 50  0001 C CNN
+	1    6600 5000
 	1    0    0    -1
 $EndComp
@@
 L power:PWR_FLAG #FLG0102
 U 1 1 5B7FBCB7
-P 5900 4700
-F 0 "#FLG0102" H 5900 4775 50  0001 C CNN
-F 1 "PWR_FLAG" H 5900 4874 50  0000 C CNN
-F 2 "" H 5900 4700 50  0001 C CNN
-F 3 "~" H 5900 4700 50  0001 C CNN
-	1    5900 4700
+P 7050 5000
+F 0 "#FLG0102" H 7050 5075 50  0001 C CNN
+F 1 "PWR_FLAG" H 7050 5174 50  0000 C CNN
+F 2 "" H 7050 5000 50  0001 C CNN
+F 3 "~" H 7050 5000 50  0001 C CNN
+	1    7050 5000
 	1    0    0    -1
 $EndComp
@@
 L power:VCC #PWR0107
 U 1 1 5B7FBCF0
-P 5900 4700
-F 0 "#PWR0107" H 5900 4550 50  0001 C CNN
-F 1 "VCC" H 5917 4873 50  0000 C CNN
-F 2 "" H 5900 4700 50  0001 C CNN
-F 3 "" H 5900 4700 50  0001 C CNN
-	1    5900 4700
+P 7050 5000
+F 0 "#PWR0107" H 7050 4850 50  0001 C CNN
+F 1 "VCC" H 7067 5173 50  0000 C CNN
+F 2 "" H 7050 5000 50  0001 C CNN
+F 3 "" H 7050 5000 50  0001 C CNN
+	1    7050 5000
 	1    0    0    1
 $EndComp
@@
 L power:GND #PWR0108
 U 1 1 5B7FBD29
-P 5450 4700
-F 0 "#PWR0108" H 5450 4450 50  0001 C CNN
-F 1 "GND" H 5455 4527 50  0000 C CNN
-F 2 "" H 5450 4700 50  0001 C CNN
-F 3 "" H 5450 4700 50  0001 C CNN
-	1    5450 4700
+P 6600 5000
+F 0 "#PWR0108" H 6600 4750 50  0001 C CNN
+F 1 "GND" H 6605 4827 50  0000 C CNN
+F 2 "" H 6600 5000 50  0001 C CNN
+F 3 "" H 6600 5000 50  0001 C CNN
+	1    6600 5000
 	1    0    0    -1
 $EndComp
@@
 	1    0    0    -1
 $EndComp
+$Comp
+L Switch:SW_Push_Dual SW?
+U 1 1 5B84D465
+P 4550 4300
+F 0 "SW?" H 4550 4585 50  0000 C CNN
+F 1 "SW_Push_Dual" H 4550 4494 50  0000 C CNN
+F 2 "" H 4550 4500 50  0001 C CNN
+F 3 "" H 4550 4500 50  0001 C CNN
+	1    4550 4300
+	1    0    0    -1
+$EndComp
+$Comp
+L Transistor_FET:IRF3205 Q?
+U 1 1 5B84D8CA
+P 4950 4300
+F 0 "Q?" H 5156 4346 50  0000 L CNN
+F 1 "IRF3205" H 5156 4255 50  0000 L CNN
+F 2 "Package_TO_SOT_THT:TO-220-3_Vertical" H 5200 4225 50  0001 L CIN
+F 3 "http://www.irf.com/product-info/datasheets/data/irf3205.pdf" H 4950 4300 50  0001 L CNN
+	1    4950 4300
+	1    0    0    -1
+$EndComp
+$Comp
+L power:GND #PWR?
+U 1 1 5B84E382
+P 5050 4500
+F 0 "#PWR?" H 5050 4250 50  0001 C CNN
+F 1 "GND" H 5055 4327 50  0000 C CNN
+F 2 "" H 5050 4500 50  0001 C CNN
+F 3 "" H 5050 4500 50  0001 C CNN
+	1    5050 4500
+	1    0    0    -1
+$EndComp
+Wire Wire Line
+	3100 3500 3650 3500
+Wire Wire Line
+	4050 3500 4350 3500
+Wire Wire Line
+	4350 3500 4350 4300
+Connection ~ 4350 3500
+Wire Wire Line
+	4350 3500 5050 3500
+Wire Wire Line
+	5050 4100 5050 3700
 $EndSCHEMATC

Commit message: Refactored circuit to use optoisolator at mosfet gate
Parts:
- removed SW?: SW_Push_Dual, symbol Switch:SW_Push_Dual
- removed U1: LM321, Package_TO_SOT_SMD:SOT-23-5, symbol Amplifier_Operational:LM321
- added C?: 2μ, symbol Device:CP
- added Q? (x2): IRF3205, Package_TO_SOT_THT:TO-220-3_Vertical, symbol Transistor_FET:IRF3205
- added Q?: 2N3906, Package_TO_SOT_THT:TO-92_Inline, symbol Transistor_BJT:2N3906
- added R? (x2): R, symbol Device:R
- added R?: 330, symbol Device:R
- added RV? (x3): R_POT, symbol Device:R_POT
- added SW?: SW_Push, symbol Switch:SW_Push
- added U? (x3): LM358, symbol Amplifier_Operational:LM358
- added U? (x2): LM321, Package_TO_SOT_SMD:SOT-23-5, symbol Amplifier_Operational:LM321
- added U?: 4N25, Package_DIP:DIP-6_W7.62mm, symbol Isolator:4N25
- C1: value CP -> 2μ
Connections:
- net labels added: Output, Output1, Output2
- wire segments 7 -> 22
Other:
- moved on the sheet: Q?
